File: esp32attachment.kicad_sch (KiCad schematic)
At the start: 36 parts, among them J1 B2B-PH-SM4-TB, J2 B2B-PH-SM4-TB, J3 B2B-PH-SM4-TB, J4 B2B-PH-SM4-TB, J5 B2B-PH-SM4-TB, J6 B2B-PH-SM4-TB, J7 BATTERY_CONNECTOR, Q1 AOD4184A, Q2 AOD4184A, Q3 AOD4184A, Q4 AOD4184A, Q5 AOD4184A, Q6 AOD4184A, U1 ESP32-DEVKIT-V1, U2 PC847, U3 PC827

Commit message: wilkkur review1 changes; still missing mounting holes
Connections:
- net FET_GATE1: now also R9.1, U2.11; no longer R7.1, U2.15
- net FET_GATE3: now also R7.1, U2.15; no longer R9.1, U2.11
- net GPIO12: now also R3.1; no longer R1.1
- net GPIO13: now also R4.1; no longer R2.1
- net GPIO14: now also R2.1; no longer R3.1
- net GPIO25: now also R1.1; no longer R4.1
Changed lines of the file:
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@@
-		)
-	)
-	(label "GPIO25"
-		(at 105.41 90.17 180)
-		(effects
-			(font
-				(size 1.27 1.27)
-			)
-			(justify right bottom)
 		)
 	)
@@
 		)
 	)
+	(label "GPIO12"
+		(at 105.41 76.2 180)
+		(effects
+			(font
+				(size 1.27 1.27)
+			)
+			(justify right bottom)
+		)
+	)
+	(label "FET_GATE3"
+		(at 137.16 53.34 180)
+		(effects
+			(font
+				(size 1.143 1.143)
+			)
+			(justify right bottom)
+		)
+	)
 	(label "FET_DRAIN6"
 		(at 167.64 133.35 180)
@@
 		)
 	)
+	(label "GPIO14"
+		(at 105.41 62.23 180)
+		(effects
+			(font
+				(size 1.27 1.27)
+			)
+			(justify right bottom)
+		)
+	)
 	(label "GPIO27"
 		(at 86.36 67.31 0)
@@
 		)
 	)
-	(label "GPIO13"
-		(at 105.41 62.23 180)
-		(effects
-			(font
-				(size 1.27 1.27)
-			)
-			(justify right bottom)
-		)
-	)
 	(label "FET_GATE6"
 		(at 162.56 140.97 180)
@@
 	)
 	(label "FET_GATE1"
+		(at 140.97 81.28 180)
+		(effects
+			(font
+				(size 1.143 1.143)
+			)
+			(justify right bottom)
+		)
+	)
+	(label "FET_GATE1"
 		(at 162.56 50.8 180)
 		(effects
 			(font
 				(size 1.143 1.143)
+			)
+			(justify right bottom)
+		)
+	)
+	(label "GPIO25"
+		(at 104.14 48.26 180)
+		(effects
+			(font
+				(size 1.27 1.27)
 			)
 			(justify right bottom)
@@
 		)
 	)
-	(label "FET_GATE3"
-		(at 140.97 81.28 180)
-		(effects
-			(font
-				(size 1.143 1.143)
-			)
-			(justify right bottom)
-		)
-	)
 	(label "FET_GATE2"
 		(at 162.56 68.58 180)
@@
 		)
 	)
-	(label "GPIO14"
-		(at 105.41 76.2 180)
-		(effects
-			(font
-				(size 1.27 1.27)
-			)
-			(justify right bottom)
-		)
-	)
-	(label "FET_GATE1"
-		(at 137.16 53.34 180)
-		(effects
-			(font
-				(size 1.143 1.143)
-			)
-			(justify right bottom)
-		)
-	)
 	(label "FET_DRAIN4"
 		(at 167.64 96.52 180)
@@
 		)
 	)
+	(label "GPIO13"
+		(at 105.41 90.17 180)
+		(effects
+			(font
+				(size 1.27 1.27)
+			)
+			(justify right bottom)
+		)
+	)
 	(label "FET_DRAIN2"
 		(at 203.2 63.5 180)
@@
 		)
 	)
-	(label "GPIO12"
-		(at 104.14 48.26 180)
-		(effects
-			(font
-				(size 1.27 1.27)
-			)
-			(justify right bottom)
-		)
-	)

Commit message: swapped out jst but need to swap it again to screw term
Parts:
- removed J1, J2, J3, J4, J5, J6: B2B-PH-SM4-TB, Connector_JST:JST_PH_B2B-PH-SM4-TB_1x02-1MP_P2.00mm_Vertical, symbol JST 2pin sidemount:B2B-PH-SM4-TB
- removed J7: BATTERY_CONNECTOR, Connector_BarrelJack:BarrelJack_Horizontal, symbol JST 2pin sidemount:B2B-PH-SM4-TB
- added J1, J2, J3, J4, J5, J6: Conn_01x02, Connector_Phoenix_SPT:PhoenixContact_SPT_1.5_2-H-3.5_1x02_P3.5mm_Horizontal, symbol Connector_Generic:Conn_01x02
- added J8: Conn_01x02, Connector_Phoenix_SPT:PhoenixContact_SPT_2.5_2-H-5.0_1x02_P5.0mm_Horizontal, symbol Connector_Generic:Conn_01x02
Connections:
- net +12V: now also J1.1 (Pin_1), J2.1 (Pin_1), J3.1 (Pin_1), J4.1 (Pin_1), J5.1 (Pin_1), J6.1 (Pin_1), J8.1 (Pin_1)
- net FET_DRAIN1: now also J1.2 (Pin_2)
- net FET_DRAIN2: now also J2.2 (Pin_2)
- net FET_DRAIN3: now also J3.2 (Pin_2)
- net FET_DRAIN4: now also J4.2 (Pin_2)
- net FET_DRAIN5: now also J5.2 (Pin_2)
- net FET_DRAIN6: now also J6.2 (Pin_2)
- net GNDPWR: now also J8.2 (Pin_2)
